File: Proto_Pi.brd (EAGLE design)
At the start: 84.8 x 56.2 mm, 32 parts, among them U1 ARDUINO_SHIELDNO_SILK

Commit message: Added PS
Parts:
- removed JP2: M20, SparkFun:1X20
- added C1: (no value), rcl:E2,5-6E
- added C2: (no value), rcl:E2,5-7
- added D1: (no value), diode:C1702-05
- added IC1: (no value), SparkFun:TO220-IGO
- added J1: POWER_JACKPTH_LOCK, SparkFun:POWER_JACK_PTH_LOCK
- added U$9: OSHW-LOGOS, SparkFun:OSHW-LOGO-S
- JP15, JP16: value M20 -> (none); device SparkFun:1X20 -> SparkFun:1X08
- JP17: device SparkFun:1X03 -> SparkFun:1X08
- JP6, JP7: value M14 -> (none); device SparkFun:1X14 -> SparkFun:1X08
- moved JP17 51.0 mm to (30.9, 2.00), turned to 90 degrees
- moved JP15 2.50 mm to (25.9, 2.00)
- moved JP16 2.50 mm to (28.4, 2.00)
- moved U1 1.00 mm to (86.0, 57.0)
Connections:
- new net 5V: C2.+, IC1.OUT, U1.5V
- new net GROUND: U$1.16
- new net N$40: C1.+, D1.C, IC1.IN
- new net N$42: D1.A, J1.PWR
- net GND: now also C1.-, C2.-, IC1.GND, J1.GND, J1.GNDBREAK, U1.GND@0; no longer U$1.16
Routing:
- net GND: track 6.63 -> 60.1 mm
- net 5V: track 0.00 -> 19.7 mm
- net N$40: track 0.00 -> 11.4 mm
- net GROUND: track 0.00 -> 7.61 mm
- net N$42: track 0.00 -> 6.27 mm
- net N$34: track 9.08 -> 7.80 mm
- net N$28: track 9.20 -> 8.00 mm
- net N$30: track 9.00 -> 7.80 mm
- net N$36: track 9.04 -> 7.90 mm
- net N$35: track 8.84 -> 7.80 mm
- net RX: track 6.51 -> 7.51 mm
- net N$33: track 8.80 -> 7.80 mm
- net N$32: track 8.50 -> 7.50 mm
- net N$31: track 8.60 -> 7.60 mm
- net N$37: track 8.90 -> 7.90 mm
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- added copper zone on layer 1, net GND
Other:
- outline, holes or cut-outs redrawn
- board text added: "Black Electronics"
- board text added: "CC-BY-SA-4.0"
- board text added: "Proto Pi"
