File: Proto_Pi.sch (EAGLE design)
At the start: 32 parts, among them U1 ARDUINO_SHIELDNO_SILK

Commit message: Added PS
Parts:
- removed JP2: M20, SparkFun:M20
- added C1: (no value), rcl:CPOL-EUE2,5-6E
- added C2: (no value), rcl:CPOL-EUE2.5-7
- added D1: (no value), diode:DIODE-C1702-05
- added IC1: (no value), SparkFun:V_REG_78XXSINK
- added J1: POWER_JACKPTH_LOCK, SparkFun:POWER_JACKPTH_LOCK
- added U$9: OSHW-LOGOS, SparkFun:OSHW-LOGOS
- JP15, JP16: value M20 -> (none); device SparkFun:M20 -> SparkFun:M081X08
- JP17: device SparkFun:M03PTH -> SparkFun:M081X08
- JP6, JP7: value M14 -> (none); device SparkFun:M14 -> SparkFun:M081X08
Connections:
- new net 5V: C2.+, IC1.OUT, U1.5V
- new net GROUND: U$1.16
- new net N$40: C1.+, D1.C, IC1.IN
- new net N$42: D1.A, J1.PWR
- net GND: now also C1.-, C2.-, IC1.GND, J1.GND, J1.GNDBREAK, U1.GND@0; no longer U$1.16
Other:
- note added: "Reference Designs ARE PROVIDED "AS IS" AND "WITH ALL FAULTS. Black Electronics DISCLAIMS ALL OTHER WARRANTIES, EXPRESS OR IMPLIED, REGARDING PRODUCTS, INCLUDING BUT NOT LIMITED TO, ANY IMPLIED WARRANTIESOF MERCHANTABILITY OR FITNESS FOR A PARTICULAR PURPOSE Black Electronics may make changes to specifications and product description at any time, without notice. The customer must not rely on the a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"
